File: hardware/mostlylevel.kicad_sch (KiCad schematic)
At the start: 27 parts, among them J1 USB-C 16P, J2 LCD QD2833 FPC, J3 CTP FT6336G FPC, J4 I2C (Qwiic), Q1 AO3400A, SW1 RESET, SW2 BOOT, U1 ESP32-S3-WROOM-1-N16R8, U2 USBLC6-2SC6, U3 ME6217C33M5G

Commit message: Hardware: reroute the PCB for revision A (#31)
The owner's KiCad work: rerouted board, updated schematic, 22 ohm series
resistors R11/R12, and the display FPC connector J2 out of the assembly
BOM. Fabrication output moves from fab/revA-draft/ to fab/revA/ (with a
Gerber zip). routing/ keeps the DRC report of each pass, the copper
layer drawings, and the board before the reroute.

The last DRC still reports 10 errors and 4 mounting holes missing from
the schematic; see the changelog.

Co-authored-by: Claude Opus 5.5 <noreply@anthropic.com>
Parts:
- added R11, R12: 22R, Resistor_SMD:R_0402_1005Metric, symbol Device:R
Connections:
- net USB_DN: now also R12.1; no longer U1.13 (USB_D-)
- net USB_DP: now also R11.1; no longer U1.14 (USB_D+)
- new net USB_DN_MCU: R12.2, U1.13 (USB_D-)
- new net USB_DP_MCU: R11.2, U1.14 (USB_D+)
